File: mpu-a/mpu-a.kicad_pcb (KiCad board)
At the start: 2 copper layers, 99.1 x 99.1 mm, 29 parts, among them J1 Conn_01x08, U1 W65C02SxP, U2 74HC245, U3 74HC00, U4 74HC245, U5 74HC245, U6 74HC245, U7 74HC138, X1 1MHz

Commit message: Specify resistors values to MPU-A
Parts:
- R10, R6, R7, R8, R9: value R -> 10K
Changed lines of the file:
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@@
         (effects (font (size 1 1) (thickness 0.15)))
     )
-    (fp_text value "R" (at 3.81 1.92 -90) (layer "F.Fab")
+    (fp_text value "10K" (at 3.81 1.92 -90) (layer "F.Fab")
         (effects (font (size 1 1) (thickness 0.15)))
     )
@@
         (effects (font (size 1 1) (thickness 0.15)))
     )
-    (fp_text value "R" (at 3.81 1.92 -90) (layer "F.Fab")
+    (fp_text value "10K" (at 3.81 1.92 -90) (layer "F.Fab")
         (effects (font (size 1 1) (thickness 0.15)))
     )
@@
         (effects (font (size 1 1) (thickness 0.15)))
     )
-    (fp_text value "R" (at 3.81 1.92 90) (layer "F.Fab")
+    (fp_text value "10K" (at 3.81 1.92 90) (layer "F.Fab")
         (effects (font (size 1 1) (thickness 0.15)))
     )
@@
         (effects (font (size 1 1) (thickness 0.15)))
     )
-    (fp_text value "R" (at 3.81 1.92 -90) (layer "F.Fab")
+    (fp_text value "10K" (at 3.81 1.92 -90) (layer "F.Fab")
         (effects (font (size 1 1) (thickness 0.15)))
     )
@@
         (effects (font (size 1 1) (thickness 0.15)))
     )
-    (fp_text value "R" (at 3.81 1.92 -90) (layer "F.Fab")
+    (fp_text value "10K" (at 3.81 1.92 -90) (layer "F.Fab")
         (effects (font (size 1 1) (thickness 0.15)))
     )
@@
     (pts (xy 101.6 60.96) (xy 200.66 60.96))
     (height -15.24)
-    (gr_text "3900.0000 mils" (at 151.13 44.57) (layer "Eco1.User")
+    (gr_text "99.0600 mm" (at 151.13 44.57) (layer "Eco1.User")
       (effects (font (size 1 1) (thickness 0.15)))
     )
@@
     (pts (xy 200.66 60.96) (xy 200.66 160.02))
     (height -30.48)
-    (gr_text "3900.0000 mils" (at 229.99 110.49 90) (layer "Eco1.User")
+    (gr_text "99.0600 mm" (at 229.99 110.49 90) (layer "Eco1.User")
       (effects (font (size 1 1) (thickness 0.15)))
     )
