File: sio-a/sio-a.kicad_sch (KiCad schematic)
At the start: 37 parts, among them J1 DE9_Plug_MountingHoles, J2 Conn_01x06, J4 Conn_02x06_Odd_Even, J5 Conn_02x06_Odd_Even, J6 Conn_02x08_Odd_Even, J7 Conn_02x08_Odd_Even, J8 Conn_02x08_Odd_Even, Q1 BC547, U1 MAX232, U3 W65C22NxP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

Commit message: Fix SIO-A CPU bus R/W logic
Connections:
- net GND: now also U2.21 (IOW); no longer U2.24 (~{IOR})
- net VCC: now also U2.24 (~{IOR}); no longer U2.21 (IOW)
Changed lines of the file:
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@@
 (kicad_sch (version 20230121) (generator eeschema)
   (paper "A4")
+  (title_block
+    (date "2023-12-28")
+    (rev "B")
+  )
   (junction (at 38.1 163.83) (diameter 0) (color 0 0 0 0)
   )
@@
     (stroke (width 0) (type default))
   )
+  (wire (pts (xy 90.17 66.04) (xy 90.17 71.12))
+    (stroke (width 0) (type default))
+  )
   (wire (pts (xy 88.9 163.83) (xy 100.33 163.83))
     (stroke (width 0) (type default))
@@
     (stroke (width 0) (type default))
   )
+  (wire (pts (xy 90.17 66.04) (xy 86.36 66.04))
+    (stroke (width 0) (type default))
+  )
   (wire (pts (xy 20.32 91.44) (xy 26.67 91.44))
     (stroke (width 0) (type default))
@@
     (stroke (width 0) (type default))
   )
-  (wire (pts (xy 91.44 71.12) (xy 104.14 71.12))
-    (stroke (width 0) (type default))
-  )
   (wire (pts (xy 139.7 110.49) (xy 143.51 110.49))
     (stroke (width 0) (type default))
@@
     (stroke (width 0) (type default))
   )
+  (wire (pts (xy 104.14 71.12) (xy 90.17 71.12))
+    (stroke (width 0) (type default))
+  )
   (wire (pts (xy 88.9 148.59) (xy 100.33 148.59))
     (stroke (width 0) (type default))
@@
     (stroke (width 0) (type default))
   )
-  (wire (pts (xy 91.44 73.66) (xy 104.14 73.66))
-    (stroke (width 0) (type default))
-  )
   (wire (pts (xy 20.32 52.07) (xy 26.67 52.07))
     (stroke (width 0) (type default))
@@
     (stroke (width 0) (type default))
   )
+  (wire (pts (xy 82.55 73.66) (xy 104.14 73.66))
+    (stroke (width 0) (type default))
+  )
   (wire (pts (xy 52.07 39.37) (xy 59.69 39.37))
     (stroke (width 0) (type default))
@@
     )
   )
-  (symbol (lib_id "power:VCC") (at 91.44 71.12 0) (unit 1)
+  (symbol (lib_id "power:VCC") (at 82.55 73.66 0) (unit 1)
     (in_bom yes) (on_board yes) (dnp no) (fields_autoplaced)
-    (property "Reference" "#PWR013" (at 91.44 74.93 0)
+    (property "Reference" "#PWR013" (at 82.55 77.47 0)
       (effects (font (size 1.27 1.27)) hide)
     )
-    (property "Value" "VCC" (at 91.44 66.04 0)
+    (property "Value" "VCC" (at 82.55 68.58 0)
       (effects (font (size 1.27 1.27)))
     )
-    (property "Footprint" "" (at 91.44 71.12 0)
+    (property "Footprint" "" (at 82.55 73.66 0)
       (effects (font (size 1.27 1.27)) hide)
     )
-    (property "Datasheet" "" (at 91.44 71.12 0)
+    (property "Datasheet" "" (at 82.55 73.66 0)
       (effects (font (size 1.27 1.27)) hide)
     )
@@
     )
   )
-  (symbol (lib_id "power:GND") (at 91.44 73.66 0) (unit 1)
+  (symbol (lib_id "power:GND") (at 86.36 66.04 0) (unit 1)
     (in_bom yes) (on_board yes) (dnp no) (fields_autoplaced)
-    (property "Reference" "#PWR014" (at 91.44 80.01 0)
+    (property "Reference" "#PWR014" (at 86.36 72.39 0)
       (effects (font (size 1.27 1.27)) hide)
     )
-    (property "Value" "GND" (at 91.44 78.74 0)
+    (property "Value" "GND" (at 86.36 71.12 0)
       (effects (font (size 1.27 1.27)))
     )
-    (property "Footprint" "" (at 91.44 73.66 0)
+    (property "Footprint" "" (at 86.36 66.04 0)
       (effects (font (size 1.27 1.27)) hide)
     )
-    (property "Datasheet" "" (at 91.44 73.66 0)
+    (property "Datasheet" "" (at 86.36 66.04 0)
       (effects (font (size 1.27 1.27)) hide)
     )

Commit message: Fix DB footprint on SCSI-A and SIO-A
Parts:
- J1: footprint Connector_Dsub:DSUB-9_Male_Horizontal_P2.77x2.84mm_EdgePinOffset4.94mm_Housed_MountingHolesOffset7.48mm -> Connector_Dsub:DSUB-9_Male_Horizontal_P2.77x2.84mm_EdgePinOffset9.90mm_Housed_MountingHolesOffset11.32mm
Changed lines of the file:
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@@
       (effects (font (size 1.27 1.27)) (justify left))
     )
-    (property "Footprint" "Connector_Dsub:DSUB-9_Male_Horizontal_P2.77x2.84mm_EdgePinOffset4.94mm_Housed_MountingHolesOffset7.48mm" (at 267.97 55.88 0)
+    (property "Footprint" "Connector_Dsub:DSUB-9_Male_Horizontal_P2.77x2.84mm_EdgePinOffset9.90mm_Housed_MountingHolesOffset11.32mm" (at 267.97 55.88 0)
       (effects (font (size 1.27 1.27)) hide)
     )
